Commit message: meta bringup implementation
Signed-off-by: Jean Laneurit <jean.laneurit@inrae.fr>

File: scout_description/urdf/scout_mini.urdf.xacro (robot description, xacro)
@@ -4,17 +4,13 @@
   <xacro:arg name="mode" default="simulation" />
   <xacro:arg name="base_name" default="base" />
-  <xacro:arg name="ros2_control_config_urdf_file" default="" />
   <xacro:arg name="controller_manager_config_yaml_file" default="" />
   <xacro:arg name="ros_prefix" default="/scout/" />
   <xacro:include filename="$(find scout_description)/urdf/scout.xacro" />
   <xacro:scout model="mini" mode="$(arg mode)" prefix="$(arg prefix)" />
-  <gazebo>
-    <plugin filename="libromea_gazebo_ros2_control.so" name="gazebo_ros2_control">
-      <ros2_control_config_file>$(arg ros2_control_config_urdf_file)</ros2_control_config_file>
-      <controller_manager_config_file>$(arg controller_manager_config_yaml_file)</controller_manager_config_file>
-      <ros>
-        <namespace>$(arg ros_prefix)$(arg base_name)</namespace>
-      </ros>
-    </plugin>
-  </gazebo>
+  <xacro:include filename="$(find scout_description)/urdf/scout.simulation.xacro" />
+  <xacro:scout_simulation
+    mode="$(arg mode)"
+    base_name="$(arg base_name)"
+    ros_prefix="$(arg ros_prefix)"
+    controller_manager_config_yaml_file="$(arg controller_manager_config_yaml_file)" />
 </robot>

File: scout_description/urdf/scout_v2.urdf.xacro (robot description, xacro)
@@ -4,17 +4,13 @@
   <xacro:arg name="mode" default="simulation" />
   <xacro:arg name="base_name" default="base" />
-  <xacro:arg name="ros2_control_config_urdf_file" default="" />
   <xacro:arg name="controller_manager_config_yaml_file" default="" />
   <xacro:arg name="ros_prefix" default="/scout/" />
   <xacro:include filename="$(find scout_description)/urdf/scout.xacro" />
   <xacro:scout model="v2" mode="$(arg mode)" prefix="$(arg prefix)" />
-  <gazebo>
-    <plugin filename="libromea_gazebo_ros2_control.so" name="gazebo_ros2_control">
-      <ros2_control_config_file>$(arg ros2_control_config_urdf_file)</ros2_control_config_file>
-      <controller_manager_config_file>$(arg controller_manager_config_yaml_file)</controller_manager_config_file>
-      <ros>
-        <namespace>$(arg ros_prefix)$(arg base_name)</namespace>
-      </ros>
-    </plugin>
-  </gazebo>
+  <xacro:include filename="$(find scout_description)/urdf/scout.simulation.xacro" />
+  <xacro:scout_simulation
+    mode="$(arg mode)"
+    base_name="$(arg base_name)"
+    ros_prefix="$(arg ros_prefix)"
+    controller_manager_config_yaml_file="$(arg controller_manager_config_yaml_file)" />
 </robot>

File: scout_description/urdf/visual/chassis.xacro (robot description, xacro)
@@ -8,5 +8,6 @@
                     rpy="0 0 ${-M_PI/2.}" />
                 <geometry>
-                    <mesh filename="package://scout_description/meshes/scout_mini_chassis.STL" />
+                    <!-- <mesh filename="package://scout_description/meshes/scout_mini_chassis.STL" /> -->
+                    <mesh filename="file://$(find scout_description)/meshes/scout_mini_chassis.STL" />
                 </geometry>
             </visual>
@@ -18,5 +19,6 @@
                     rpy="0 0 0" />
                 <geometry>
-                    <mesh filename="package://scout_description/meshes/scout_v2_chassis.dae" />
+                    <!-- <mesh filename="package://scout_description/meshes/scout_v2_chassis.dae" /> -->
+                    <mesh filename="file://$(find scout_description)/meshes/scout_v2_chassis.dae" />
                 </geometry>
             </visual>
