Commit message: [description] update ros2 control xacro file
Signed-off-by: Jean Laneurit <jean.laneurit@inrae.fr>

File: scout_description/ros2_control/scout.ros2_control.xacro (robot description, xacro)
@@ -35,16 +35,32 @@
     <xacro:property name="maximal_wheel_speed"
       value="${props['wheels_speed_control']['command']['maximal_speed']}" />
-    <!-- hardware plugins -->
-    <xacro:property name="simulation_hardware_plugin"
-      value="romea_mobile_base_gazebo/GazeboSystemInterface4WD" />
-    <xacro:if value="${model == 'mini'}">
-      <xacro:property name="live_hardware_plugin"
-        value="scout_hardware/ScoutMiniHardware" />
+    <xacro:if value="${mode == 'simulation_gazebo'}">
+      <xacro:property
+        name="hardware_plugin"
+        value="romea_mobile_base_gazebo/GazeboSystemInterface" />
     </xacro:if>
-    <xacro:if value="${model == 'v2'}">
-      <xacro:property name="live_hardware_plugin"
-        value="scout_hardware/ScoutV2Hardware" />
+    <xacro:if value="${mode == 'simulation_gazebo_classic'}">
+        <xacro:property name="hardware_plugin"
+          value="campero_hardware/GazeboSystemInterface4WD" />
     </xacro:if>
-    <xacro:base_control mode="${mode}" base_name="${base_name}" />
+    <xacro:if value="${'4dv' in mode or 'isaac' in mode}">
+      <xacro:property
+        name="hardware_plugin"
+        value="romea_mobile_base_simulation/GenericSimulationSystemInterface" />
+    </xacro:if>
+    <xacro:if value="${mode ==  'live'}">
+      <xacro:if value="${model == 'mini'}">
+        <xacro:property name="hardware_plugin"
+          value="scout_hardware/ScoutMiniHardware" />
+      </xacro:if>
+      <xacro:if value="${model == 'v2'}">
+        <xacro:property name="hardware_plugin"
+          value="scout_hardware/ScoutV2Hardware" />
+      </xacro:if>
+    </xacro:if>
+    <xacro:base_control
+      mode="${mode}"
+      base_name="${base_name}"
+      hardware_plugin="${hardware_plugin}" />
   </xacro:macro>
 </robot>

Commit message: [description] add scout_properties.xacro
Signed-off-by: Jean Laneurit <jean.laneurit@inrae.fr>

File: scout_description/ros2_control/scout.ros2_control.xacro (robot description, xacro)
@@ -2,37 +2,7 @@
 <robot name="scout_ros2_control" xmlns:xacro="http://www.ros.org/wiki/xacro">
   <xacro:macro name="scout_ros2_control" params="mode model prefix base_name">
-    <xacro:include
-      filename="$(find romea_mobile_base_description)/ros2_control/base4WD.ros2_control.xacro" />
+    <xacro:include filename="$(find romea_mobile_base_description)/ros2_control/base4WD.ros2_control.xacro" />
     <xacro:property name="conf" value="$(find scout_description)/config/scout_${model}.yaml" />
-    <xacro:property name="props" value="${load_yaml(conf)}" />
-    <!-- Joint names -->
-    <xacro:property name="base_footprint_joint"
-      value="${props['joints']['base_footprint_joint_name']}" />
-    <xacro:property name="inertial_joint" value="${props['joints']['inertial_joint_name']}" />
-    <xacro:property name="front_left_wheel_spinning_joint"
-      value="${props['joints']['front_left_wheel_spinning_joint_name']}" />
-    <xacro:property name="front_right_wheel_spinning_joint"
-      value="${props['joints']['front_right_wheel_spinning_joint_name']}" />
-    <xacro:property name="rear_left_wheel_spinning_joint"
-      value="${props['joints']['rear_left_wheel_spinning_joint_name']}" />
-    <xacro:property name="rear_right_wheel_spinning_joint"
-      value="${props['joints']['rear_right_wheel_spinning_joint_name']}" />
-    <!-- Geometry -->
-    <xacro:property name="wheelbase"
-      value="${props['geometry']['axles_distance']}" />
-    <xacro:property name="front_track"
-      value="${props['geometry']['front_axle']['wheels_distance']}" />
-    <xacro:property name="rear_track"
-      value="${props['geometry']['rear_axle']['wheels_distance']}" />
-    <xacro:property name="front_wheel_radius"
-      value="${props['geometry']['front_axle']['wheels']['radius']}" />
-    <xacro:property name="rear_wheel_radius"
-      value="${props['geometry']['rear_axle']['wheels']['radius']}" />
-    <xacro:property name="front_hub_carrier_offset"
-      value="${props['geometry']['front_axle']['wheels']['hub_carrier_offset']}" />
-    <xacro:property name="rear_hub_carrier_offset"
-      value="${props['geometry']['rear_axle']['wheels']['hub_carrier_offset']}" />
-    <xacro:property name="maximal_wheel_speed"
-      value="${props['wheels_speed_control']['command']['maximal_speed']}" />
+    <xacro:include filename="$(find scout_description)/urdf/scout_properties.xacro" />
     <xacro:if value="${mode == 'simulation_gazebo'}">
       <xacro:property

File: scout_description/urdf/scout.xacro (robot description, xacro)
@@ -7,97 +7,5 @@
       <xacro:include filename="$(find scout_description)/urdf/visual/wheels.xacro" />
       <xacro:property name="conf" value="$(find scout_description)/config/scout_${model}.yaml" />
-      <xacro:property name="props" value="${load_yaml(conf)}" />
-      <!-- Link names -->
-      <xacro:property name="base_link"
-         value="${props['links']['base_link_name']}" />
-      <xacro:property name="base_footprint_link"
-         value="${props['links']['base_footprint_link_name']}" />
-      <xacro:property name="inertial_link"
-         value="${props['links']['inertial_link_name']}" />
-      <xacro:property name="front_left_wheel_spinning_link"
-         value="${props['links']['front_left_wheel_spinning_link_name']}" />
-      <xacro:property name="front_right_wheel_spinning_link"
-         value="${props['links']['front_right_wheel_spinning_link_name']}" />
-      <xacro:property name="rear_left_wheel_spinning_link"
-         value="${props['links']['rear_left_wheel_spinning_link_name']}" />
-      <xacro:property name="rear_right_wheel_spinning_link"
-         value="${props['links']['rear_right_wheel_spinning_link_name']}" />
-      <!-- Joint names -->
-      <xacro:property name="base_footprint_joint"
-         value="${props['joints']['base_footprint_joint_name']}" />
-      <xacro:property name="inertial_joint"
-         value="${props['joints']['inertial_joint_name']}" />
-      <xacro:property name="front_left_wheel_spinning_joint"
-         value="${props['joints']['front_left_wheel_spinning_joint_name']}" />
-      <xacro:property name="front_right_wheel_spinning_joint"
-         value="${props['joints']['front_right_wheel_spinning_joint_name']}" />
-      <xacro:property name="rear_left_wheel_spinning_joint"
-         value="${props['joints']['rear_left_wheel_spinning_joint_name']}" />
-      <xacro:property name="rear_right_wheel_spinning_joint"
-         value="${props['joints']['rear_right_wheel_spinning_joint_name']}" />
-      <!-- Base Properties -->
-      <xacro:property name="aabb_length"
-         value="${props['geometry']['aabb']['length']}" />
-      <xacro:property name="aabb_width"
-         value="${props['geometry']['aabb']['width']}" />
-      <xacro:property name="aabb_height"
-         value="${props['geometry']['aabb']['height']}" />
-      <xacro:property name="aabb_center_x"
-         value="${props['geometry']['aabb']['center'][0]}" />
-      <xacro:property name="aabb_center_y"
-         value="${props['geometry']['aabb']['center'][1]}" />
-      <xacro:property name="aabb_center_z"
-         value="${props['geometry']['aabb']['center'][2]}" />
-      <xacro:property name="wheelbase"
-         value="${props['geometry']['axles_distance']}" />
-      <xacro:property name="front_track"
-         value="${props['geometry']['front_axle']['wheels_distance']}" />
-      <xacro:property name="rear_track"
-         value="${props['geometry']['rear_axle']['wheels_distance']}" />
-      <xacro:property name="track"
-         value="${front_track}" />
-      <xacro:property name="ground_clearance"
-         value="${chassis_props['ground_clearance']}" />
-      <xacro:property name="mass_body"
-         value="${props['inertia']['mass']}" />
-      <xacro:property name="mass_base"
-         value="${props['inertia']['mass']}" />
-      <xacro:property name="mass_center_x"
-         value="${props['inertia']['center'][0]}" />
-      <xacro:property name="mass_center_y"
-         value="${props['inertia']['center'][1]}" />
-      <xacro:property name="mass_center_z"
-         value="${props['inertia']['center'][2]}" />
-      <xacro:property name="ground_clearance"
-         value="${props['geometry']['ground_clearance']}" />
-      <xacro:property name="body_reference_x"
-         value="${props['control_point'][0]}" />
-      <!-- Steering Properties -->
-      <xacro:property name="front_wheel_y_offset"
-         value="${props['geometry']['front_axle']['wheels']['hub_carrier_offset']}" />
-      <xacro:property name="rear_wheel_y_offset"
-         value="${props['geometry']['rear_axle']['wheels']['hub_carrier_offset']}" />
-      <xacro:property name="wheel_y_offset"
-         value="${front_wheel_y_offset}" />
-      <!-- Wheel Properties -->
-      <xacro:property name="front_hub_carrier_offset"
-         value="${props['geometry']['front_axle']['wheels']['hub_carrier_offset']}" />
-      <xacro:property name="rear_hub_carrier_offset"
-         value="${props['geometry']['rear_axle']['wheels']['hub_carrier_offset']}" />
-      <xacro:property name="front_wheel_radius"
-         value="${props['geometry']['front_axle']['wheels']['radius']}" />
-      <xacro:property name="rear_wheel_radius"
-         value="${props['geometry']['rear_axle']['wheels']['radius']}" />
-      <xacro:property name="front_wheel_width"
-         value="${props['geometry']['front_axle']['wheels']['width']}" />
-      <xacro:property name="rear_wheel_width"
-         value="${props['geometry']['rear_axle']['wheels']['width']}" />
-      <xacro:property name="maximal_wheel_speed"
-         value="${props['wheels_speed_control']['command']['maximal_speed']}" />
-      <xacro:property name="wheel_mass" value="5" />
-      <xacro:property name="front_wheel_mass" value="5" />
-      <xacro:property name="rear_wheel_mass" value="5" />
-      <xacro:property name="chassis_height"
-         value="${min(front_wheel_radius,rear_wheel_radius)}" />
+      <xacro:include filename="$(find scout_description)/urdf/scout_properties.xacro" />
       <xacro:chassis>
          <chassis_visuals>
